Commit message: added gripper

File: robinion_description/urdf/robinion.structure.arm.xacro (robot description, xacro)
@@ -138,4 +138,30 @@
 		<link name="l_wrist">
 		</link>
+		<joint name="l_gripper_fixed_joint" type="fixed">
+			<parent link="l_arm_3_link"/>
+			<child link="l_gripper"/>
+			<origin xyz="0.000 0.068 -0.025" rpy="0 0 0"/>
+		</joint>
+		<link name="l_gripper">
+			<collision>
+				<origin xyz="0.00 0.00 0.00" rpy="0.00 0.00 0.00"/>
+				<geometry>
+					<mesh filename="package://robinion_description/meshes/collision/l_gripper_collision.stl"/>
+				</geometry>
+			</collision>
+			<visual>
+				<origin xyz="0.00 0.00 0.00" rpy="0.00 0.00 0.00"/>
+				<geometry>
+					<mesh filename="package://robinion_description/meshes/visual/l_gripper_visual.stl"/>
+				</geometry>
+			</visual>
+			<inertial>
+				<origin xyz="0.000000 0.043774 0.003216" rpy="0.00 0.00 0.00"/>
+				<mass value="0.247773"/>
+				<inertia ixx="0.000210" ixy="0.000000" ixz="0.000000"
+						 iyy="0.000119" iyz="0.000017"
+						 izz="0.000219" />
+			</inertial>
+		</link>
 	</xacro:macro>
 	<xacro:macro name="robinion_r_arm" params="parent">
@@ -275,4 +301,30 @@
 		<link name="r_wrist">
 		</link>
+		<joint name="r_gripper_fixed_joint" type="fixed">
+			<parent link="r_arm_3_link"/>
+			<child link="r_gripper"/>
+			<origin xyz="0.000 -0.068 -0.025" rpy="0 0 0"/>
+		</joint>
+		<link name="r_gripper">
+			<collision>
+				<origin xyz="0.00 0.00 0.00" rpy="0.00 0.00 0.00"/>
+				<geometry>
+					<mesh filename="package://robinion_description/meshes/collision/r_gripper_collision.stl"/>
+				</geometry>
+			</collision>
+			<visual>
+				<origin xyz="0.00 0.00 0.00" rpy="0.00 0.00 0.00"/>
+				<geometry>
+					<mesh filename="package://robinion_description/meshes/visual/r_gripper_visual.stl"/>
+				</geometry>
+			</visual>
+			<inertial>
+				<origin xyz="0.000000 -0.043774 0.003216" rpy="0.00 0.00 0.00"/>
+				<mass value="0.247773"/>
+				<inertia ixx="0.000210" ixy="0.000000" ixz="0.000000"
+						 iyy="0.000119" iyz="-0.000017"
+						 izz="0.000219" />
+			</inertial>
+		</link>
 	</xacro:macro>
 </robot>

Commit message: fix inverted joint in real robot

File: robinion_description/urdf/robinion.structure.arm.xacro (robot description, xacro)
@@ -39,5 +39,5 @@
 			<child link="l_arm_1_link"/>
 			<origin xyz="0.025 0.033 -0.021" rpy="0 0 0"/>
-			<axis xyz="1 0 0"/>
+			<axis xyz="-1 0 0"/>
 			<limit velocity="3.14" effort="10.6" lower="${-pi*0.5}" upper="${pi*0.5}" />
 			<!-- <limit velocity="3.14" effort="100" lower="-3" upper="3" /> -->
@@ -103,5 +103,5 @@
 			<child link="l_arm_3_link"/>
 			<origin xyz="0.022 0.060 0.025" rpy="0 0 0"/>
-			<axis xyz="0 0 1"/>
+			<axis xyz="0 0 -1"/>
 			<limit velocity="3.14" effort="10.6" lower="${-pi*0.5}" upper="${pi*0.5}" />
 			<!-- <limit velocity="3.14" effort="100" lower="-3" upper="3" /> -->
@@ -153,5 +153,5 @@
 				<origin xyz="0.00 0.00 0.00" rpy="0.00 0.00 0.00"/>
 				<geometry>
-					<mesh filename="package://robinion_description/meshes/visual/l_gripper_visual.stl"/>
+					<mesh filename="package://robinion_description/meshes/visual/l_gripper_closed_visual.stl"/>
 				</geometry>
 			</visual>
@@ -163,4 +163,11 @@
 						 izz="0.000219" />
 			</inertial>
+		</link>
+		<joint name="l_end_effector_fixed_joint" type="fixed">
+			<parent link="l_gripper"/>
+			<child link="l_end_effector"/>
+			<origin xyz="0.000 0.1 0.0" rpy="0 0 0"/>
+		</joint>
+		<link name="l_end_effector">
 		</link>
 	</xacro:macro>
@@ -170,5 +177,5 @@
 			<child link="r_shoulder_link"/>
 			<origin xyz="-0.021 -0.131 0.139" rpy="0 0 0"/>
-			<axis xyz="0 1 0"/>
+			<axis xyz="0 -1 0"/>
 			<limit velocity="3.14" effort="10.6" lower="${-pi*0.9}" upper="${pi*0.9}" />
 			<!-- <limit velocity="3.14" effort="100" lower="-3" upper="3" /> -->
@@ -202,5 +209,5 @@
 			<child link="r_arm_1_link"/>
 			<origin xyz="0.025 -0.033 -0.021" rpy="0 0 0"/>
-			<axis xyz="1 0 0"/>
+			<axis xyz="-1 0 0"/>
 			<limit velocity="3.14" effort="10.6" lower="${-pi*0.5}" upper="${pi*0.5}" />
 			<!-- <limit velocity="3.14" effort="100" lower="-3" upper="3" /> -->
@@ -234,5 +241,5 @@
 			<child link="r_arm_2_link"/>
 			<origin xyz="-0.025 -0.118 0.000" rpy="0 0 0"/>
-			<axis xyz="0 1 0"/>
+			<axis xyz="0 -1 0"/>
 			<limit velocity="4.82" effort="4.1" lower="${-pi*0.9}" upper="${pi*0.9}" />
 			<!-- <limit velocity="4.82" effort="100" lower="-3" upper="3" /> -->
@@ -266,5 +273,5 @@
 			<child link="r_arm_3_link"/>
 			<origin xyz="0.022 -0.060 0.025" rpy="0 0 0"/>
-			<axis xyz="0 0 1"/>
+			<axis xyz="0 0 -1"/>
 			<limit velocity="3.14" effort="10.6" lower="${-pi*0.5}" upper="${pi*0.5}" />
 			<!-- <limit velocity="3.14" effort="100" lower="-3" upper="3" /> -->
@@ -316,5 +323,5 @@
 				<origin xyz="0.00 0.00 0.00" rpy="0.00 0.00 0.00"/>
 				<geometry>
-					<mesh filename="package://robinion_description/meshes/visual/r_gripper_visual.stl"/>
+					<mesh filename="package://robinion_description/meshes/visual/r_gripper_closed_visual.stl"/>
 				</geometry>
 			</visual>
@@ -327,4 +334,11 @@
 			</inertial>
 		</link>
+		<joint name="r_end_effector_fixed_joint" type="fixed">
+			<parent link="r_gripper"/>
+			<child link="r_end_effector"/>
+			<origin xyz="0.000 -0.1 0.0" rpy="0 0 0"/>
+		</joint>
+		<link name="r_end_effector">
+		</link>
 	</xacro:macro>
 </robot>

File: robinion_description/urdf/robinion.structure.head.xacro (robot description, xacro)
@@ -39,5 +39,5 @@
 			<child link="head_pitch_link"/>
 			<origin xyz="0.000 0.019 0.047" rpy="0 0 0"/>
-			<axis xyz="0 1 0"/>
+			<axis xyz="0 -1 0"/>
 			<limit velocity="4.82" effort="4.1" lower="${-pi*0.5}" upper="${pi*0.5}" />
 			<!-- <limit velocity="4.82" effort="1000" lower="-3" upper="3" /> -->

File: robinion_description/urdf/robinion.structure.leg.xacro (robot description, xacro)
@@ -7,5 +7,5 @@
 			<child link="l_hip_yaw_link"/>
 			<origin xyz="0.000 0.055 -0.006" rpy="0 0 0"/>
-			<axis xyz="0 0 1"/>
+			<axis xyz="0 0 -1"/>
 			<limit velocity="3.14" effort="10.6" lower="${-pi*0.9}" upper="${pi*0.9}" />
 			<!-- <limit velocity="3.14" effort="100" lower="-3" upper="3" /> -->
@@ -39,5 +39,5 @@
 			<child link="l_hip_roll_pitch_link"/>
 			<origin xyz="0.048 0.000 -0.051" rpy="0 0 0"/>
-			<axis xyz="1 0 0"/>
+			<axis xyz="-1 0 0"/>
 			<limit velocity="4.08" effort="9.90" lower="${-pi*0.25}" upper="${pi*0.25}" />
 			<!-- <limit velocity="4.08" effort="100" lower="-3" upper="3" /> -->
@@ -253,5 +253,5 @@
 			<child link="l_ankle_roll_pitch_link"/>
 			<origin xyz="0.000 0.000 -0.200" rpy="0 0 0"/>
-			<axis xyz="0 1 0"/>
+			<axis xyz="0 -1 0"/>
 			<limit velocity="4.08" effort="9.90" lower="${-pi*0.5}" upper="${pi*0.5}" />
 			<!-- <limit velocity="4.08" effort="100" lower="-3" upper="3" /> -->
@@ -349,5 +349,5 @@
 			<child link="r_hip_yaw_link"/>
 			<origin xyz="0.000 -0.055 -0.006" rpy="0 0 0"/>
-			<axis xyz="0 0 1"/>
+			<axis xyz="0 0 -1"/>
 			<limit velocity="3.14" effort="10.6" lower="${-pi*0.9}" upper="${pi*0.9}" />
 			<!-- <limit velocity="3.14" effort="1000" lower="-3" upper="3" /> -->
@@ -381,5 +381,5 @@
 			<child link="r_hip_roll_pitch_link"/>
 			<origin xyz="0.048 0.000 -0.051" rpy="0 0 0"/>
-			<axis xyz="1 0 0"/>
+			<axis xyz="-1 0 0"/>
 			<limit velocity="4.08" effort="9.90" lower="${-pi*0.25}" upper="${pi*0.25}" />
 			<!-- <limit velocity="4.08" effort="100" lower="-3" upper="3" /> -->
@@ -413,5 +413,5 @@
 			<child link="r_thigh_back_link"/>
 			<origin xyz="-0.066 0.025 0.000" rpy="0 0 0"/>
-			<axis xyz="0 1 0"/>
+			<axis xyz="0 -1 0"/>
 			<limit velocity="4.08" effort="9.90" lower="${-pi*0.5}" upper="${pi*0.5}" />
 			<!-- <limit velocity="4.08" effort="100" lower="-3" upper="3" /> -->
